Commit message: increased rotation speed of camera

File: cob_description/ros/urdf/head_v1/head.urdf.xacro (robot description, xacro)
@@ -18,5 +18,5 @@
 			<dynamics damping="0.1" />
 			<calibration rising="${head_axis_ref}"/>
-			<limit effort="100" lower="-3.2" upper="0.1" velocity="0.5"/>
+			<limit effort="100" lower="-3.2" upper="0.1" velocity="1.0"/>
 		</joint>
 		<link name="${name}_axis_link">

Commit message: adapted tf of kinect

File: cob_description/ros/urdf/head_v1/head.urdf.xacro (robot description, xacro)
@@ -50,5 +50,5 @@
 		<!-- cam3d -->
 		<xacro:cob_kinect_v0 name="${name}_cam3d" ros_topic="cam3d/depth/points1" parent="${name}_color_camera_l_link">
-			<origin xyz="${cam3d_x-0.06} ${cam3d_y} ${cam3d_z}" rpy="${cam3d_roll} ${cam3d_pitch} ${cam3d_yaw+3.14}" />
+			<origin xyz="${cam3d_x-0.06} ${cam3d_y-0.05} ${cam3d_z}" rpy="${cam3d_roll+0.05} ${cam3d_pitch} ${cam3d_yaw+3.14}" />
 		</xacro:cob_kinect_v0>
 		<!-- extensions -->

Commit message: increased upper limit of head axis

File: cob_description/ros/urdf/head_v1/head.urdf.xacro (robot description, xacro)
@@ -18,5 +18,5 @@
 			<dynamics damping="0.1" />
 			<calibration rising="${head_axis_ref}"/>
-			<limit effort="100" lower="-3.2" upper="0.1" velocity="1.0"/>
+			<limit effort="100" lower="-3.2" upper="0.25" velocity="1.0"/>
 		</joint>
 		<link name="${name}_axis_link">
