Commit message: update the kinect to hand calibration

File: cob_description/ros/calibration/cob3-1.urdf.xacro (robot description, xacro)
@@ -36,9 +36,9 @@
 	<property name="cam_r_yaw" value="0.00676" />
 	<!-- cam3d to left calibration -->
-	<property name="cam3d_x" value="0.0" />
-	<property name="cam3d_y" value="0.0" />
-	<property name="cam3d_z" value="0.0" />
-	<property name="cam3d_roll" value="0.0" />
-	<property name="cam3d_pitch" value="0.0" />
-	<property name="cam3d_yaw" value="0.0" />
+	<property name="cam3d_x" value="-0.07188823" />
+	<property name="cam3d_y" value="-0.03216233" />
+	<property name="cam3d_z" value="-0.07915284" />
+	<property name="cam3d_roll" value="0.03" />
+	<property name="cam3d_pitch" value="0.01078" />
+	<property name="cam3d_yaw" value="-0.00241" />
 </robot>

File: cob_description/ros/urdf/head_v1/head.urdf.xacro (robot description, xacro)
@@ -50,5 +50,5 @@
 		<!-- cam3d -->
 		<xacro:cob_kinect_v0 name="${name}_cam3d" ros_topic="cam3d/depth/points1" parent="${name}_color_camera_l_link">
-			<origin xyz="${cam3d_x-0.06} ${cam3d_y-0.05} ${cam3d_z}" rpy="${cam3d_roll+0.05} ${cam3d_pitch} ${cam3d_yaw+3.14}" />
+			<origin xyz="${cam3d_x} ${cam3d_y} ${cam3d_z}" rpy="${cam3d_roll} ${cam3d_pitch} ${cam3d_yaw+3.14}" />
 		</xacro:cob_kinect_v0>
 		<!-- extensions -->
