Commit message: update kinect mounting pose for cob3-1

File: cob_description/urdf/head_v1/head.urdf.xacro (robot description, xacro)
@@ -42,5 +42,5 @@
 		<!-- left camera -->
 		<xacro:cob_prosilica_v0 name="${name}_color_camera_l" ros_topic="stereo/left" parent="${name}_axis_link">
-			<origin xyz="${cam_l_x} ${cam_l_y} ${cam_l_z-0.06}" rpy="${cam_l_roll} ${cam_l_pitch+M_PI/2} ${cam_l_yaw+M_PI}" />
+			<origin xyz="${cam_l_x} ${cam_l_y} ${cam_l_z-0.06}" rpy="${cam_l_roll} ${cam_l_pitch+M_PI/2} ${cam_l_yaw}" />
 		</xacro:cob_prosilica_v0>
 		<!-- right camera -->
@@ -50,5 +50,5 @@
 		<!-- cam3d -->
 		<xacro:cob_kinect_v0 name="${name}_cam3d" ros_topic="cam3d" parent="${name}_color_camera_l_link">
-			<origin xyz="${cam3d_x-0.06} ${cam3d_y} ${cam3d_z}" rpy="${cam3d_roll} ${cam3d_pitch} ${cam3d_yaw}" />
+			<origin xyz="${cam3d_x-0.06} ${cam3d_y} ${cam3d_z}" rpy="${cam3d_roll} ${cam3d_pitch} ${cam3d_yaw+M_PI}" />
 		</xacro:cob_kinect_v0>
 		<!-- extensions -->

Commit message: revert back to old head_v1 version

File: cob_description/urdf/head_v1/head.urdf.xacro (robot description, xacro)
@@ -42,5 +42,5 @@
 		<!-- left camera -->
 		<xacro:cob_prosilica_v0 name="${name}_color_camera_l" ros_topic="stereo/left" parent="${name}_axis_link">
-			<origin xyz="${cam_l_x} ${cam_l_y} ${cam_l_z-0.06}" rpy="${cam_l_roll} ${cam_l_pitch+M_PI/2} ${cam_l_yaw}" />
+			<origin xyz="${cam_l_x} ${cam_l_y} ${cam_l_z-0.06}" rpy="${cam_l_roll} ${cam_l_pitch+M_PI/2} ${cam_l_yaw+M_PI}" />
 		</xacro:cob_prosilica_v0>
 		<!-- right camera -->
@@ -50,5 +50,5 @@
 		<!-- cam3d -->
 		<xacro:cob_kinect_v0 name="${name}_cam3d" ros_topic="cam3d" parent="${name}_color_camera_l_link">
-			<origin xyz="${cam3d_x-0.06} ${cam3d_y} ${cam3d_z}" rpy="${cam3d_roll} ${cam3d_pitch} ${cam3d_yaw+M_PI}" />
+			<origin xyz="${cam3d_x-0.06} ${cam3d_y} ${cam3d_z}" rpy="${cam3d_roll} ${cam3d_pitch} ${cam3d_yaw}" />
 		</xacro:cob_kinect_v0>
 		<!-- extensions -->
