Commit message: revert torso limit fixes

File: cob_description/urdf/torso_v0/torso.urdf.xacro (robot description, xacro)
@@ -25,5 +25,5 @@
       <calibration rising="${torso_lower_neck_pan_ref}"/>
       <dynamics damping="25.0" friction="10.0"/>
-      <limit effort="24" lower="-0.1" upper="0.1" velocity="0.5"/>
+      <limit effort="24" lower="-1.0" upper="1.0" velocity="0.5"/>
     </joint>
     <link name="${name}_lower_neck_pan_link">
@@ -55,5 +55,5 @@
       <dynamics damping="25.0" friction="10.0"/>
       <calibration rising="${torso_lower_neck_tilt_ref}"/>
-      <limit effort="46" lower="-0.25" upper="0.25" velocity="0.5"/>
+      <limit effort="46" lower="-0.4" upper="0.4" velocity="0.5"/>
     </joint>
     <link name="${name}_lower_neck_tilt_link">
@@ -85,5 +85,5 @@
       <dynamics damping="25.0" friction="10.0"/>
       <calibration rising="${torso_upper_neck_pan_ref}"/>
-      <limit effort="4" lower="-0.2" upper="0.2" velocity="0.5"/>
+      <limit effort="4" lower="-1.0" upper="1.0" velocity="0.5"/>
     </joint>
     <link name="${name}_upper_neck_pan_link">
@@ -115,5 +115,5 @@
       <dynamics damping="25.0" friction="10.0"/>
       <calibration rising="${torso_upper_neck_tilt_ref}"/>
-      <limit effort="24" lower="-0.3" upper="0.3" velocity="0.5"/>
+      <limit effort="24" lower="-0.4" upper="0.4" velocity="0.5"/>
     </joint>
     <link name="${name}_upper_neck_tilt_link">
