Commit message: [cob3-1] change the upper limit for the head axis

File: cob_description/urdf/cob3_head/head_prosilicas_kinect.urdf.xacro (robot description, xacro)
@@ -34,5 +34,5 @@
       <axis xyz="0 0 1" />
       <dynamics damping="0.1" />
-      <limit effort="100" lower="-3.2" upper="0.1" velocity="1.4"/>
+      <limit effort="100" lower="-3.54" upper="0.1" velocity="1.4"/>
     </joint>
     <link name="${name}_axis_link">
