Commit message: increase velocity and limits of upper neck pan and tilt

File: cob_description/urdf/cob3_torso/torso_v1.urdf.xacro (robot description, xacro)
@@ -85,5 +85,5 @@
       <dynamics damping="25.0" friction="10.0"/>
       <calibration rising="${torso_upper_neck_pan_ref}"/>
-      <limit effort="200" lower="-1.0" upper="1.0" velocity="0.5"/>
+      <limit effort="200" lower="-1.5" upper="1.5" velocity="1.0"/>
     </joint>
     <link name="${name}_upper_neck_pan_link">
@@ -115,5 +115,5 @@
       <dynamics damping="25.0" friction="10.0"/>
       <calibration rising="${torso_upper_neck_tilt_ref}"/>
-      <limit effort="200" lower="-0.4" upper="0.4" velocity="0.5"/>
+      <limit effort="200" lower="-0.65" upper="0.95" velocity="1.0"/>
     </joint>
     <link name="${name}_upper_neck_tilt_link">

Commit message: increase torso limits to allow initialization

File: cob_description/urdf/cob3_torso/torso_v1.urdf.xacro (robot description, xacro)
@@ -32,5 +32,5 @@
       <axis xyz="0 0 1" />
       <dynamics damping="25.0" friction="10.0"/>
-      <limit effort="200" lower="-0.1" upper="0.1" velocity="0.5"/>
+      <limit effort="200" lower="-0.6" upper="0.6" velocity="0.5"/>
     </joint>
     <link name="${name}_lower_neck_pan_link">
@@ -91,5 +91,5 @@
       <axis xyz="0 0 1" />
       <dynamics damping="25.0" friction="10.0"/>
-      <limit effort="200" lower="-0.2" upper="0.2" velocity="0.5"/>
+      <limit effort="200" lower="-1.1" upper="1.1" velocity="0.5"/>
     </joint>
     <link name="${name}_upper_neck_pan_link">

Commit message: [robocup 2016] extreme torso and gripper bounding box

File: cob_description/urdf/cob3_torso/torso_v1.urdf.xacro (robot description, xacro)
@@ -61,5 +61,5 @@
       <axis xyz="0 0 1" />
       <dynamics damping="25.0" friction="10.0"/>
-      <limit effort="200" lower="-0.26" upper="0.25" velocity="0.5"/>
+      <limit effort="200" lower="-0.26" upper="0.90" velocity="0.5"/>
     </joint>
     <link name="${name}_lower_neck_tilt_link">
@@ -120,5 +120,5 @@
       <axis xyz="0 0 1" />
       <dynamics damping="25.0" friction="10.0"/>
-      <limit effort="200" lower="-0.21" upper="0.3" velocity="0.5"/>
+      <limit effort="200" lower="-0.21" upper="0.9" velocity="0.5"/>
     </joint>
     <link name="${name}_upper_neck_tilt_link">

File: cob_description/urdf/lbr/lbr.urdf.xacro (robot description, xacro)
@@ -247,4 +247,24 @@
       </collision>
     </link>
+    <!-- joint between arm_7_link and arm_gripper_box -->
+    <joint name="${name}_gripper_box_joint" type="fixed">
+      <origin xyz="0 -0.01 0.17" rpy="0 0 0" />
+      <parent link="${name}_7_link"/>
+      <child link="${name}_gripper_box_link"/>
+    </joint>
+    <link name="${name}_gripper_box_link">
+      <visual>
+        <origin xyz="0 0 0" rpy="0 0 0" />
+        <geometry>
+          <box size="0.12 0.18 0.15"/>
+        </geometry>
+      </visual>
+      <collision>
+        <origin xyz="0 0 0" rpy="0 0 0" />
+        <geometry>
+          <box size="0.12 0.18 0.15"/>
+        </geometry>
+      </collision>
+    </link>
     <!-- extensions -->
     <xacro:lbr_gazebo name="${name}" />
